Commit message: 3D 激光雷达，但是还不正常，rslidar_mems

File: summit_xl_common-melodic/summit_xl_description/robots/summit_xl_gen_std.urdf.xacro (robot description, xacro)
@@ -74,7 +74,7 @@
         </xacro:sensor_hokuyo_ust10lx-->
         <!-- 3d laser -->
-        <!--xacro:sensor_rslidar_mems prefix="$(arg prefix)top_3d_laser" parent="$(arg prefix)base_link">
+        <xacro:sensor_rslidar_mems prefix="$(arg prefix)top_3d_laser" parent="$(arg prefix)base_link">
             <origin xyz="0.3134 0 0.2424" rpy="0 0 0"/>
-        </xacro:sensor_rslidar_mems-->
+        </xacro:sensor_rslidar_mems>
         <!-- ptz camera -->
         <!--xacro:sensor_axis prefix="$(arg prefix)front_ptz_camera" parent="$(arg prefix)base_link">

File: summit_xl_common-melodic/summit_xl_description/robots/summit_xl_std.urdf.xacro (robot description, xacro)
@@ -63,7 +63,14 @@
 		</xacro:sensor_imu>
 		<!-- 2d laser -->
-		<xacro:sensor_hokuyo_ust10lx prefix="$(arg prefix)front_laser" parent="$(arg prefix)base_link" prefix_topic="front_laser" gpu="$(arg gpu)">
+		<!-- <xacro:sensor_hokuyo_ust10lx prefix="$(arg prefix)front_laser" parent="$(arg prefix)base_link" prefix_topic="front_laser" gpu="$(arg gpu)">
 			<origin xyz="0.0 0.0 0.33" rpy="0 0 0"/>
-		</xacro:sensor_hokuyo_ust10lx>
+		</xacro:sensor_hokuyo_ust10lx> -->
+		<!-- 3d laser -->
+		<!-- <xacro:sensor_hokuyo3d prefix="$(arg prefix)front_laser" parent="$(arg prefix)base_link" prefix_topic="front_laser" gpu="$(arg gpu)">
+			<origin xyz="0.0 0.0 0.33" rpy="0 0 0"/>
+		</xacro:sensor_hokuyo3d> -->
+		<xacro:sensor_rslidar_mems prefix="$(arg prefix)top_3d_laser" parent="$(arg prefix)base_link">
+            <origin xyz="0.3134 0 0.2424" rpy="0 0 0"/>
+        </xacro:sensor_rslidar_mems>
 		<!-- ptz camera -->
 		<xacro:sensor_axis prefix="$(arg prefix)front_ptz_camera" parent="$(arg prefix)base_link">
