Commit message: vrlodyne 3D激光可以，hokuyo不行？

File: summit_xl_common-melodic/summit_xl_description/robots/summit_xl_std.urdf.xacro (robot description, xacro)
@@ -19,5 +19,6 @@
 	<!-- Flag to select the high or low quality model -->
 	<xacro:property name="hq" value="true" />
-	<xacro:arg name="prefix" default="summit_xl_"/>
+	<!-- <xacro:arg name="prefix" default="summit_xl_"/> -->
+	<xacro:arg name="prefix" default="robot_"/>
 	<xacro:arg name="ros_planar_move_plugin" default="false"/>
 	<xacro:arg name="omni_wheels" default="false"/>
@@ -67,12 +68,16 @@
 		</xacro:sensor_hokuyo_ust10lx>
 		<!-- 3d laser -->
-		<xacro:sensor_hokuyo3d prefix="$(arg prefix)3d_laser" parent="$(arg prefix)base_link"  gpu="$(arg gpu)">
-			<origin xyz="0.0 0.0 0.33" rpy="0 0 0"/>
-		</xacro:sensor_hokuyo3d>
-        <!-- <xacro:sensor_velodyne_vlp16 prefix="$(arg prefix)_3d_laser" parent="$(arg prefix)base_link"  gpu="$(arg gpu)" >
-            <origin xyz="0.3134 0 0.2424" rpy="0 0 0"/>
-			<range_min  />
-			<range_max  />
-        </xacro:sensor_velodyne_vlp16> -->
+		<!-- <xacro:sensor_hokuyo3d prefix="$(arg prefix)3d_laser" parent="$(arg prefix)base_link"  gpu="$(arg gpu)">
+			<origin xyz="0.1 0.1 0.53" rpy="1.57 0 0"/>
+		</xacro:sensor_hokuyo3d> -->
+		  <!-- <xacro:include filename="$(find velodyne_description)/urdf/VLP-16.urdf.xacro"/> -->
+  <!-- <xacro:VLP-16 parent="$(arg prefix)base_link" name="velodyne" topic="/velodyne_points" hz="10" samples="440" gpu="${gpu}">
+    <origin xyz="0 0 0.4" rpy="0 0 0" />
+  </xacro:VLP-16> -->
+        <xacro:sensor_velodyne_vlp16 prefix="$(arg prefix)3d_laser" parent="$(arg prefix)base_link" range_min = "0.9" range_max="130.0" gpu="$(arg gpu)" >
+            <origin xyz="0.3134 0 0.5424" rpy="0 0 0"/>
+			<!-- <range_min  />
+			<range_max  /> -->
+        </xacro:sensor_velodyne_vlp16>
 		<!-- ptz camera -->
 		<xacro:sensor_axis prefix="$(arg prefix)front_ptz_camera" parent="$(arg prefix)base_link">

Commit message: 添加pid yaml参数正常控制，但是rviz显示不正常

File: summit_xl_common-melodic/summit_xl_description/robots/summit_xl_std.urdf.xacro (robot description, xacro)
@@ -9,5 +9,5 @@
 	<!-- Import summit XL wheels -->
 	<xacro:include filename="$(find summit_xl_description)/urdf/wheels/rubber_wheel.urdf.xacro" />
-  <xacro:include filename="$(find summit_xl_description)/urdf/wheels/omni_wheel.urdf.xacro" />
+  <!-- <xacro:include filename="$(find summit_xl_description)/urdf/wheels/omni_wheel.urdf.xacro" /> -->
 	<!-- Import all available sensors -->
 	<xacro:include filename="$(find robotnik_sensors)/urdf/all_sensors.urdf.xacro" />
@@ -19,9 +19,9 @@
 	<!-- Flag to select the high or low quality model -->
 	<xacro:property name="hq" value="true" />
-	<!-- <xacro:arg name="prefix" default="summit_xl_"/> -->
-	<xacro:arg name="prefix" default="robot_"/>
+	<xacro:arg name="prefix" default="summit_xl_"/>
+	<!-- <xacro:arg name="prefix" default="robot_"/> -->
 	<xacro:arg name="ros_planar_move_plugin" default="false"/>
 	<xacro:arg name="omni_wheels" default="false"/>
-	<xacro:arg name="gpu" default="false"/>
+	<xacro:arg name="gpu" default="true"/>
     <xacro:macro name="summit_xl" params="prefix publish_bf hq">
 		<!-- *************** -->
@@ -75,8 +75,6 @@
     <origin xyz="0 0 0.4" rpy="0 0 0" />
   </xacro:VLP-16> -->
-        <xacro:sensor_velodyne_vlp16 prefix="$(arg prefix)3d_laser" parent="$(arg prefix)base_link" range_min = "0.9" range_max="130.0" gpu="$(arg gpu)" >
-            <origin xyz="0.3134 0 0.5424" rpy="0 0 0"/>
-			<!-- <range_min  />
-			<range_max  /> -->
+        <xacro:sensor_velodyne_vlp16 prefix="$(arg prefix)3d_laser" parent="$(arg prefix)base_link"  range_min = "0.9" range_max="130.0" gpu="$(arg gpu)" >
+            <origin xyz="0.3134 0.0 0.5424" rpy="0 0 0"/>
         </xacro:sensor_velodyne_vlp16>
 		<!-- ptz camera -->

Commit message: x

File: summit_xl_common-melodic/summit_xl_description/robots/summit_xl_std.urdf.xacro (robot description, xacro)
@@ -63,14 +63,20 @@
 		</xacro:sensor_imu>
 		<!-- 2d laser -->
-		<xacro:sensor_hokuyo_ust10lx prefix="$(arg prefix)front_laser" parent="$(arg prefix)base_link" prefix_topic="front_laser" gpu="$(arg gpu)">
+		<!-- <xacro:sensor_hokuyo_ust10lx prefix="$(arg prefix)front_laser" parent="$(arg prefix)base_link" prefix_topic="front_laser" gpu="$(arg gpu)">
 			<origin xyz="0.0 0.0 0.33" rpy="0 0 0"/>
-		</xacro:sensor_hokuyo_ust10lx>
+		</xacro:sensor_hokuyo_ust10lx> -->
 		<!-- 3d laser -->
 		<!-- <xacro:sensor_hokuyo3d prefix="$(arg prefix)front_laser" parent="$(arg prefix)base_link" prefix_topic="front_laser" gpu="$(arg gpu)">
 			<origin xyz="0.0 0.0 0.33" rpy="0 0 0"/>
 		</xacro:sensor_hokuyo3d> -->
-        <xacro:sensor_hokuyo3d prefix="$(arg prefix)top_3d_laser" parent="$(arg prefix)base_link">
-            <origin xyz="0.3134 0 0.2424" rpy="0 0 0"/>
-        </xacro:sensor_hokuyo3d>
+        <!-- <xacro:sensor_velodyne_vlp16 prefix="$(arg prefix)threed_laser" parent="$(arg prefix)base_link" range_min="0.9" range_max="130.0">
+            <origin xyz="0.3134 0 0.5424" rpy="0 0 0"/>
+        </xacro:sensor_velodyne_vlp16> -->
+		      <!-- <xacro:sensor_rslidar_mems prefix="$(arg prefix)top_3d_laser" parent="$(arg prefix)base_link">
+        <origin xyz="0.3134 0 0.2424" rpy="0 0 0"/>
+      </xacro:sensor_rslidar_mems> -->
+	          <xacro:sensor_rslidar_16 prefix="$(arg prefix)top_3d_laser" parent="$(arg prefix)base_link">
+            <origin xyz="-0.2776 0 0.629" rpy="0 0 0"/>
+        </xacro:sensor_rslidar_16>
 		<!-- ptz camera -->
 		<xacro:sensor_axis prefix="$(arg prefix)front_ptz_camera" parent="$(arg prefix)base_link">
