Commit message: 模型3d数据正常

File: summit_xl_common/summit_xl_description/robots/sxl_std.urdf.xacro (robot description, xacro)
@@ -64,9 +64,9 @@
 		<!-- 2d laser -->
 		<xacro:sensor_hokuyo_ust10lx prefix="$(arg prefix)front_laser" parent="$(arg prefix)base_link" prefix_topic="front_laser" gpu="$(arg gpu)">
-			<origin xyz="0.0 0.0 0.33" rpy="0 0 0"/>
+			<origin xyz="0.0 0.0 0.3" rpy="0 0 0"/>
 		</xacro:sensor_hokuyo_ust10lx>
 		<!-- 3d laser -->
 		<xacro:sensor_velodyne_vlp16 prefix="$(arg prefix)top_laser" parent="$(arg prefix)base_link" prefix_topic="top_laser" range_min="0.9" range_max="130" gpu="$(arg gpu)">
-			<origin xyz="0.0 0.0 0.45" rpy="0 0 0"/>
+			<origin xyz="0.0 0.0 0.4" rpy="0 0 0"/>
 		</xacro:sensor_velodyne_vlp16>
 		        <!-- <xacro:sensor_rslidar_mems prefix="$(arg prefix)top_3d_laser" parent="$(arg prefix)base_link">
