Commit message: vins 不正常，里程计飘了

File: summit_xl_common/summit_xl_description/robots/sxl_std_3d.urdf.xacro (robot description, xacro)
@@ -63,7 +63,7 @@
 		</xacro:sensor_imu>
 		<!-- 2d laser -->
-		<xacro:sensor_hokuyo_ust10lx prefix="$(arg prefix)front_laser" parent="$(arg prefix)base_link" prefix_topic="front_laser" gpu="$(arg gpu)">
+		<!-- <xacro:sensor_hokuyo_ust10lx prefix="$(arg prefix)front_laser" parent="$(arg prefix)base_link" prefix_topic="front_laser" gpu="$(arg gpu)">
 			<origin xyz="0.0 0.0 0.3" rpy="0 0 0"/>
-		</xacro:sensor_hokuyo_ust10lx>
+		</xacro:sensor_hokuyo_ust10lx> -->
 		<!-- 3d laser -->
 		<xacro:sensor_velodyne_vlp16 prefix="$(arg prefix)top_laser" parent="$(arg prefix)base_link" prefix_topic="top_laser" range_min="0.9" range_max="130" gpu="$(arg gpu)">
@@ -78,11 +78,7 @@
 		</xacro:sensor_axis>
 	  <!-- RGBD -->
-	  	<!-- <xacro:sensor_orbbec_astra prefix="$(arg prefix)front_rgbd_camera" parent="$(arg prefix)base_link" prefix_topic="front_rgbd_camera">
+	  <xacro:sensor_orbbec_astra prefix="$(arg prefix)front_rgbd_camera" parent="$(arg prefix)base_link" prefix_topic="front_rgbd_camera">
 			<origin xyz="0.324 0.012 0.172" rpy="0 0 0"/>
-		</xacro:sensor_orbbec_astra> -->
-		<!-- zed -->
-		<xacro:stereolabs_zed prefix="$(arg prefix)front_zed_camera" parent="$(arg prefix)base_link" >
-			<origin xyz="0.324 0.012 0.172" rpy="0 0 0"/>
-		</xacro:stereolabs_zed>
+		</xacro:sensor_orbbec_astra>
 	  <!-- GPS -->
 	  <xacro:sensor_gps prefix="$(arg prefix)gps" parent="$(arg prefix)base_link" gps_latitude="$(arg gps_latitude)" gps_longitude="$(arg gps_longitude)">

File: summit_xl_common/summit_xl_description/robots/sxl_std_stereo.urdf.xacro (robot description, xacro)
@@ -67,7 +67,7 @@
 		</xacro:sensor_hokuyo_ust10lx>
 		<!-- 3d laser -->
-		<xacro:sensor_velodyne_vlp16 prefix="$(arg prefix)top_laser" parent="$(arg prefix)base_link" prefix_topic="top_laser" range_min="0.9" range_max="130" gpu="$(arg gpu)">
+		<!-- <xacro:sensor_velodyne_vlp16 prefix="$(arg prefix)top_laser" parent="$(arg prefix)base_link" prefix_topic="top_laser" range_min="0.9" range_max="130" gpu="$(arg gpu)">
 			<origin xyz="0.0 0.0 0.4" rpy="0 0 0"/>
-		</xacro:sensor_velodyne_vlp16>
+		</xacro:sensor_velodyne_vlp16> -->
 		        <!-- <xacro:sensor_rslidar_mems prefix="$(arg prefix)top_3d_laser" parent="$(arg prefix)base_link">
             <origin xyz="0.3134 0 0.2424" rpy="0 0 0"/>
@@ -78,9 +78,13 @@
 		</xacro:sensor_axis>
 	  <!-- RGBD -->
-	  	<!-- <xacro:sensor_orbbec_astra prefix="$(arg prefix)front_rgbd_camera" parent="$(arg prefix)base_link" prefix_topic="front_rgbd_camera">
+	  <!-- <xacro:sensor_orbbec_astra prefix="$(arg prefix)front_rgbd_camera" parent="$(arg prefix)base_link" prefix_topic="front_rgbd_camera">
 			<origin xyz="0.324 0.012 0.172" rpy="0 0 0"/>
 		</xacro:sensor_orbbec_astra> -->
+		<!-- ???? -->
+	  <!-- <xacro:stereo_camera prefix="$(arg prefix)front_rgbd_camera" parent="$(arg prefix)base_link" prefix_topic="front_rgbd_camera">
+			<origin xyz="0.324 0.012 0.172" rpy="0 0 0"/>
+		</xacro:stereo_camera> -->
 		<!-- zed -->
-		<xacro:stereolabs_zed prefix="$(arg prefix)front_zed_camera" parent="$(arg prefix)base_link" >
+	  <xacro:stereolabs_zed prefix="$(arg prefix)front_zed_camera" parent="$(arg prefix)base_link" >
 			<origin xyz="0.324 0.012 0.172" rpy="0 0 0"/>
 		</xacro:stereolabs_zed>
