Commit message: x

File: summit_xl_common/summit_xl_description/robots/summit_xl_std.urdf.xacro (robot description, xacro)
@@ -66,4 +66,14 @@
 			<origin xyz="0.0 0.0 0.33" rpy="0 0 0"/>
 		</xacro:sensor_hokuyo_ust10lx>
+		<!-- 3d laser  -->
+		<xacro:sensor_velodyne_vlp16 prefix="$(arg prefix)top_laser" parent="$(arg prefix)base_link"  range_min="-2.3562" range_max="2.3562" gpu="$(arg gpu)">
+			<origin xyz="0.0 0.0 0.33" rpy="0 0 0"/>
+		</xacro:sensor_velodyne_vlp16>
+		<!-- <xacro:sensor_rslidar_mems prefix="$(arg prefix)top_3d_laser" parent="$(arg prefix)base_link">
+			<origin xyz="0.3134 0 0.2424" rpy="0 0 0"/>
+		</xacro:sensor_rslidar_mems> -->
+				<!-- <xacro:sensor_sick_s300 prefix="$(arg prefix)rear_laser" parent="$(arg prefix)base_link" prefix_topic="rear_laser" gpu="$(arg gpu)">
+			<origin xyz="${rear_laser_offset_x} ${rear_laser_offset_y} ${rear_laser_offset_z}" rpy="0 ${-PI} ${-1/4*PI}" />
+		</xacro:sensor_sick_s300> -->
 		<!-- ptz camera -->
 		<xacro:sensor_axis prefix="$(arg prefix)front_ptz_camera" parent="$(arg prefix)base_link">

Commit message: 源代码程序初次运行

File: summit_xl_common/summit_xl_description/robots/summit_xl_std.urdf.xacro (robot description, xacro)
@@ -9,5 +9,5 @@
 	<!-- Import summit XL wheels -->
 	<xacro:include filename="$(find summit_xl_description)/urdf/wheels/rubber_wheel.urdf.xacro" />
-  <!-- <xacro:include filename="$(find summit_xl_description)/urdf/wheels/omni_wheel.urdf.xacro" /> -->
+  <xacro:include filename="$(find summit_xl_description)/urdf/wheels/omni_wheel.urdf.xacro" />
 	<!-- Import all available sensors -->
 	<xacro:include filename="$(find robotnik_sensors)/urdf/all_sensors.urdf.xacro" />
@@ -20,8 +20,7 @@
 	<xacro:property name="hq" value="true" />
 	<xacro:arg name="prefix" default="summit_xl_"/>
-	<!-- <xacro:arg name="prefix" default="robot_"/> -->
 	<xacro:arg name="ros_planar_move_plugin" default="false"/>
 	<xacro:arg name="omni_wheels" default="false"/>
-	<xacro:arg name="gpu" default="true"/>
+	<xacro:arg name="gpu" default="false"/>
     <xacro:macro name="summit_xl" params="prefix publish_bf hq">
 		<!-- *************** -->
@@ -67,17 +66,4 @@
 			<origin xyz="0.0 0.0 0.33" rpy="0 0 0"/>
 		</xacro:sensor_hokuyo_ust10lx>
-		<!-- 3d laser -->
-		<!-- <xacro:sensor_hokuyo3d prefix="$(arg prefix)3d_laser" parent="$(arg prefix)base_link"  gpu="$(arg gpu)">
-			<origin xyz="0.1 0.1 0.53" rpy="1.57 0 0"/>
-		</xacro:sensor_hokuyo3d> -->
-		  <!-- <xacro:include filename="$(find velodyne_description)/urdf/VLP-16.urdf.xacro"/> -->
-  <!-- <xacro:VLP-16 parent="$(arg prefix)base_link" name="velodyne" topic="/velodyne_points" hz="10" samples="440" gpu="${gpu}">
-    <origin xyz="0 0 0.4" rpy="0 0 0" />
-  </xacro:VLP-16> -->
-        <xacro:sensor_velodyne_vlp16 prefix="$(arg prefix)3d_laser" parent="$(arg prefix)base_link" range_min = "0.9" range_max="130.0" gpu="$(arg gpu)" >
-            <origin xyz="0.3134 0 0.5424" rpy="0 0 0"/>
-			<!-- <range_min  />
-			<range_max  /> -->
-        </xacro:sensor_velodyne_vlp16>
 		<!-- ptz camera -->
 		<xacro:sensor_axis prefix="$(arg prefix)front_ptz_camera" parent="$(arg prefix)base_link">

File: summit_xl_common/summit_xl_description/robots/summit_xls_std.urdf.xacro (robot description, xacro)
@@ -43,5 +43,4 @@
 	<xacro:property name="hq" value="true" />
 	<xacro:arg name="prefix" default="summit_xl_"/>
-	<!-- <xacro:arg name="prefix" default="robot_"/> -->
 	<xacro:arg name="ros_planar_move_plugin" default="false"/>
 	<xacro:arg name="gpu" default="false"/>

File: summit_xl_common/summit_xl_description/urdf/bases/summit_xl_base.urdf.xacro (robot description, xacro)
@@ -7,5 +7,4 @@
 	  <xacro:property name="wheel_radius" value="0.11"/>
 	  <!-- BASE FOOTPRINT -->
-	  <!-- prefix 参数 就是: robot_ -->
 	  <xacro:if value="${publish_bf}">
 		<link name="${prefix}base_footprint">
